Commit message: simplify meshes

File: urdf/stompy_pro/robot.urdf (robot description, URDF)
Before this commit: robot robot, 22 links, 21 joints
Links:
- added link base_2, mass 0.001
- added link base_2_2, mass 0.001
Joints:
- added joint floating_base_2: type fixed, parent base_2_2, child base_2_2, origin xyz=0 0 0 rpy=0 0 0
- added joint floating_base_2_2: type fixed, parent base_2_2, child trunk, origin xyz=0 0 0.0 rpy=0 0 0
- joint floating_base: child trunk -> base_2; origin xyz=0 0 0.0 rpy=0 0 0 -> xyz=0 0 0 rpy=0 0 0; parent base -> base_2

Commit message: simplified teleop

File: urdf/stompy_pro/robot.urdf (robot description, URDF)
Before this commit: robot robot, 24 links, 23 joints
Links:
- removed link L_buttock
- removed link L_calf
- removed link L_foot
- removed link L_leg
- removed link L_thigh
- removed link R_buttock
- removed link R_calf
- removed link R_foot
- removed link R_leg
- removed link R_thigh
- removed link base_2
- removed link base_2_2
Joints:
- removed joint L_ankle_y
- removed joint L_hip_x
- removed joint L_hip_y
- removed joint L_hip_z
- removed joint L_knee
- removed joint R_ankle_y
- removed joint R_hip_x
- removed joint R_hip_y
- removed joint R_hip_z
- removed joint R_knee
- removed joint floating_base_2
- removed joint floating_base_2_2
- joint floating_base: child base_2 -> trunk; origin xyz=0 0 0 rpy=0 0 0 -> xyz=0 0 0.0 rpy=0 0 0; parent base_2 -> base

Commit message: smoothing

File: urdf/stompy_pro/robot.urdf (robot description, URDF)
Before this commit: robot robot, 12 links, 11 joints
Joints:
- joint left_end_effector_joint: origin xyz=-.05 0 -.1 rpy=0 0 0 -> xyz=-0.05 0 -0.1 rpy=0 0 0
- joint right_end_effector_joint: origin xyz=-.05 0 -.1 rpy=0 0 0 -> xyz=-0.05 0 -0.1 rpy=0 0 0
